Commit message: Fix duplicate materials.xacro include

File: src/my_bot/description/robot_core.xacro (robot description, xacro)
@@ -1,4 +1,16 @@
 <?xml version="1.0"?>
 <robot xmlns:xacro="http://www.ros.org/wiki/xacro">
+    <xacro:property name="chassis_radius" value="0.155"/>
+    <xacro:property name="chassis_length" value="0.065"/>
+    <xacro:property name="chassis_mass" value="1.5"/>
+    <xacro:property name="chassis_offset_z" value="0.0325"/>
+    <xacro:property name="wheel_radius" value="0.0325"/>
+    <xacro:property name="wheel_thickness" value="0.012"/>
+    <xacro:property name="wheel_mass" value="0.05"/>
+    <xacro:property name="wheel_offset_y" value="0.160"/>
+    <xacro:property name="wheel_offset_z" value="-0.010"/>
+    <xacro:property name="caster_wheel_radius" value="0.010"/>
+    <xacro:property name="caster_wheel_mass" value="0.02"/>
+    <xacro:property name="caster_wheel_offset_x" value="0.038"/>
     <xacro:include filename="inertial_macros.xacro"/>
     <material name="white">
@@ -134,143 +146,2 @@
     </link>
 </robot>
-<!--<?xml version="1.0"?>
-<robot xmlns:xacro="http://www.ros.org/wiki/xacro">
-    <xacro:include filename="inertial_macros.xacro"/>
-    <material name="white">
-        <color rgba="1 1 1 1"/>
-    </material>
-    <material name="blue">
-        <color rgba="0.2 0.2 1 1"/>
-    </material>
-    <material name="black">
-        <color rgba="0 0 0 1"/>
-    </material>
-     <material name="dark_grey">
-        <color rgba="0.3 0.3 0.3 1"/>
-    </material>
-    <material name="red">
-        <color rgba="0.2 0.2 1 1"/>
-    </material>
-- Base link" على اﻻرض-
-    <link name="base_link"/>
-- Chassis link في نص الجسم -
-    <joint name="chassis_joint" type="fixed">
-        <parent link="base_link"/>
-        <child link="chassis"/>
-        <origin xyz="0 0 0.0325"/>
-    </joint>
-    <link name="chassis">
-        <visual>
-            <origin xyz="0.0 0.0 0.0" rpy="0.0 0.0 0.0"/>
-            <geometry>
-                <cylinder radius="0.155" length="0.065"/>
-            </geometry>
-            <material name="black"/>
-        </visual>
-        <collision>
-            <origin xyz="0.0 0.0 0.0" rpy="0.0 0.0 0.0"/>
-            <geometry>
-                <cylinder radius="0.155" length="0.065"/>
-            </geometry>
-        </collision>
-        <xacro:inertial_cylinder mass="1.5" length="0.065" radius="0.155">
-          <origin xyz="0 0 0" rpy="0 0 0"/>
-        </xacro:inertial_cylinder>
-    </link>
-- LEFT wheel -
-    <joint name="left_wheel_joint" type="continuous">
-        <parent link="chassis"/>
-        <child link="left_wheel"/>
-        <origin xyz="0 0.160 -0.010" rpy="-1.5707 0 0"/>
-        <axis xyz="0 0 1"/>
-    </joint>
-    <link name="left_wheel">
-      <visual>
-        <geometry>
-            <cylinder radius="0.0325" length="0.012"/>
-        </geometry>
-        <material name="dark_grey"/>
-      </visual>
-      <collision>
-        <geometry>
-            <cylinder radius="0.0325" length="0.012"/>
-        </geometry>
-      </collision>
-      <xacro:inertial_cylinder mass="0.05" length="0.012" radius="0.0325">
-        <origin xyz="0 0 0" rpy="0 0 0"/>
-      </xacro:inertial_cylinder>
-    </link>
-- RIGHT wheel -
-    <joint name="right_wheel_joint" type="continuous">
-        <parent link="chassis"/>
-        <child link="right_wheel"/>
-        <origin xyz="0 -0.160 -0.010" rpy="-1.5707 0 0"/>
-        <axis xyz="0 0 1"/>
-    </joint>
-  <link name="right_wheel">
-    <visual>
-        <origin xyz="0 0 0" rpy="0 0 0"/>
-        <geometry>
-            <cylinder radius="0.0325" length="0.012"/>
-        </geometry>
-        <material name="dark_grey"/>
-    </visual>
-    <collision>
-        <origin xyz="0 0 0" rpy="0 0 0"/>
-        <geometry>
-            <cylinder radius="0.0325" length="0.012"/>
-        </geometry>
-    </collision>
-    <xacro:inertial_cylinder mass="0.05" length="0.012" radius="0.0325">
-        <origin xyz="0 0 0" rpy="0 0 0"/>
-    </xacro:inertial_cylinder>
-  </link>
-- RIGHT CASTER wheel -
- <joint name="right_caster_joint" type="fixed">
-    <parent link="base_link"/>
-    <child link="right_caster_link"/>
-    <origin xyz="0.038 0.0 0.0" rpy="0.0 0.0 0.0"/>
- </joint>
- <link name="right_caster_link">
-  <visual>
-    <origin xyz="0.038 0.0 0.0" rpy="0.0 0.0 0.0"/>
-    <geometry>
-        <sphere radius="0.010"/>
-    </geometry>
-    <material name="white"/>
-  </visual>
-  <collision>
-    <origin xyz="0.038 0.0 0.0" rpy="0.0 0.0 0.0"/>
-    <geometry>
-        <sphere radius="0.010"/>
-    </geometry>
-  </collision>
-  <xacro:inertial_sphere mass="0.02" radius="0.020">
-     <origin xyz="0.038 0.0 0.0" rpy="0 0 0"/>
-  </xacro:inertial_sphere>
- </link>
-- LEFT CASTER wheel -
- <joint name="left_caster_joint" type="fixed">
-    <parent link="base_link"/>
-    <child link="left_caster_link"/>
-    <origin xyz="-0.038 0.0 0.0" rpy="0.0 0.0 0.0"/>
- </joint>
- <link name="left_caster_link">
-  <visual>
-    <origin xyz="-0.038 0.0 0.0" rpy="0.0 0.0 0.0"/>
-    <geometry>
-        <sphere radius="0.010"/>
-    </geometry>
-    <material name="white"/>
-  </visual>
-  <collision>
-    <origin xyz="-0.038 0.0 0.0" rpy="0.0 0.0 0.0"/>
-    <geometry>
-        <sphere radius="0.010"/>
-    </geometry>
-  </collision>
-  <xacro:inertial_sphere mass="0.02" radius="0.020">
-     <origin xyz="0.038 0.0 0.0" rpy="0 0 0"/>
-  </xacro:inertial_sphere>
- </link>
-</robot> -->
