Commit message: Pi: single laser_frame in lidar.xacro, add base_footprint

File: src/my_bot/description/lidar.xacro (robot description, xacro)
@@ -70,66 +70,2 @@
     </gazebo>
 </robot>
-<!--<?xml version="1.0"?>
-<robot xmlns:xacro="http://www.ros.org/wiki/xacro">
-    <material name="red">
-       <color rgba="0.2 0.2 1 1"/>
- </material>
- <joint name="laser_joint" type="fixed">
-    <parent link="chassis"/>
-    <child link="laser_frame"/>
-    <origin xyz="0.0 0.0 0.05" rpy="0.0 0.0 0.0"/>
- </joint>
- <link name="laser_frame">
-  <visual>
-    <geometry>
-        <cylinder radius="0.0325" length="0.012"/>
-    </geometry>
-    <material name="red"/>
-  </visual>
-  <collision>
-    <geometry>
-        <cylinder radius="0.0325" length="0.012"/>
-    </geometry>
-  </collision>
-  <xacro:inertial_cylinder mass="0.01" length="0.012" radius="0.0325">
-    <origin xyz="0 0 0" rpy="0 0 0"/>
-  </xacro:inertial_cylinder>
- </link>
- <gazebo reference="laser_frame">
-    <material>Gazebo/Red</material>
-    <sensor name="lidar" type="gpu_lidar">
-        <pose relative_to="lidar_link"> 0 0 0 0 0 0</pose>
-        <topic>scan</topic>
-        <visualize>true</visualize>
-        <update_rate>10</update_rate>
-        <always_on>true</always_on>
-        <gz_frame_id>lidar_link</gz_frame_id>
-        <lidar>
-            <scan>
-                <horizontal>
-                    <samples>720</samples>
-                    <resolution>1</resolution>
-                    <min_angle>-3.14159</min_angle>
-                    <max_angle>3.14159</max_angle>
-                </horizontal>
-                <vertical>
-                    <samples>1</samples>
-                    <resolution>1</resolution>
-                    <min_angle>0</min_angle>
-                    <max_angle>0</max_angle>
-                </vertical>
-            </scan>
-            <range>
-                <min>0.1</min>
-                <max>12.0</max>
-                <resolution>0.01</resolution>
-            </range>
-            <noise>
-                <type>gaussian</type>
-                <mean>0.0</mean>
-                <stddev>0.01</stddev>
-            </noise>
-        </lidar>
-    </sensor>
- </gazebo>
-</robot> -->

File: src/my_bot/description/robot_core.xacro (robot description, xacro)
@@ -28,4 +28,11 @@
     <!-- Base link: ground reference frame -->
     <link name="base_link"/>
+    <!-- BASE_FOOTPRINT LINK-->
+    <joint name="base_footprint_joint" type="fixed">
+        <parent link="base_link"/>
+        <child link="base_footprint"/>
+        <origin xyz="0 0 0" rpy="0 0 0"/>
+    </joint>
+    <link name="base_footprint"/>
     <!-- Chassis -->
     <joint name="chassis_joint" type="fixed">
